Commit message: Working slam and bringup. Nav not working correctly

File: src/kmr_description/urdf/kmp200/kmp200.xacro (robot description, xacro)
@@ -40,7 +40,9 @@
       <parent link="base_link"/>
       <child link="base_footprint"/>
+      <origin rpy="0 0 0.0" xyz="0 0 0"/>
+    </joint>
+    <link name="base_footprint">
       <origin rpy="0 0 0.0" xyz="0 0 -${ground_clearance}"/>
-    </joint>
-    <link name="base_footprint"/>
+    </link>
     <joint name="${robot_name}_base_link_to_top" type="fixed">
       <parent link="base_link"/>

File: src/kmr_description/urdf/robot/kmr_simple_camera_wo_wheels.urdf (robot description, URDF)
Before this commit: robot kmr, 36 links, 35 joints
Joints:
- joint kmr_footprint_to_base_link: origin xyz=0 0 -0.025 rpy=0 0 0.0 -> xyz=0 0 0 rpy=0 0 0.0
